File: unnamedpcb.kicad_pcb (KiCad board)
At the start: 2 copper layers, 0 parts

Commit message: Updated FIles
Parts:
- added C1: 100n, Capacitor_SMD:C_0402_1005Metric, F.Cu at (92.8, 55.8)
- added C10: 10p, Capacitor_SMD:C_0402_1005Metric, F.Cu at (87.5, 60.8)
- added C11: 10p, Capacitor_SMD:C_0402_1005Metric, F.Cu at (87.5, 62.8)
- added C12: 22u, Capacitor_SMD:C_0805_2012Metric, F.Cu at (104.0, 64.5)
- added C13: 22u, Capacitor_SMD:C_0805_2012Metric, F.Cu at (108.8, 70.0)
- added C2: 100n, Capacitor_SMD:C_0402_1005Metric, F.Cu at (101.2, 59.2)
- added C3: 100n, Capacitor_SMD:C_0402_1005Metric, F.Cu at (97.8, 67.8)
- added C4: 100n, Capacitor_SMD:C_0402_1005Metric, F.Cu at (89.2, 58.5)
- added C5: 10u, Capacitor_SMD:C_0603_1608Metric, F.Cu at (92.8, 52.8)
- added C6: 10n, Capacitor_SMD:C_0402_1005Metric, F.Cu at (89.2, 62.8)
- added C7: 1u, Capacitor_SMD:C_0402_1005Metric, F.Cu at (88.5, 66.5)
- added C8: 1u, Capacitor_SMD:C_0402_1005Metric, F.Cu at (88.5, 68.0)
- added C9: 100n, Capacitor_SMD:C_0402_1005Metric, F.Cu at (93.0, 68.0)
- added D1: RED, LED_SMD:LED_0603_1608Metric, F.Cu at (113.0, 70.0)
- added FB1: 120R, Inductor_SMD:L_0603_1608Metric, F.Cu at (90.2, 67.2)
- added H1: MountingHole, MountingHole:MountingHole_2.2mm_M2, F.Cu at (79.2, 42.5)
- added H2: MountingHole, MountingHole:MountingHole_2.2mm_M2, F.Cu at (116.0, 42.5)
- added H3: MountingHole, MountingHole:MountingHole_2.2mm_M2, F.Cu at (79.2, 75.0)
- added H4: MountingHole, MountingHole:MountingHole_2.2mm_M2, F.Cu at (116.5, 75.0)
- added J1: USB_B_Micro, Connector_USB:USB_Micro-B_Wuerth_629105150521, F.Cu at (110.0, 60.0)
- added J2: Conn_01x04_Pin, Connector_PinHeader_1.27mm:PinHeader_1x04_P1.27mm_Vertical, F.Cu at (102.0, 45.8)
- added J3: Conn_01x04_Pin, Connector_PinHeader_1.27mm:PinHeader_1x04_P1.27mm_Vertical, F.Cu at (95.4, 45.8)
- added J4: Conn_01x04_Pin, Connector_PinHeader_1.27mm:PinHeader_1x04_P1.27mm_Vertical, F.Cu at (94.1, 73.0)
- added R1: 10k, Resistor_SMD:R_0402_1005Metric, F.Cu at (88.5, 48.8)
- added R2: 1k5, Resistor_SMD:R_0402_1005Metric, F.Cu at (104.8, 59.5)
- added R3: 1k5, Resistor_SMD:R_0402_1005Metric, F.Cu at (113.0, 67.2)
- added R4: 1k5, Resistor_SMD:R_0402_1005Metric, F.Cu at (94.6, 70.8)
- added R5: 1k5, Resistor_SMD:R_0402_1005Metric, F.Cu at (96.8, 70.8)
- added SW1: SW_SPDT, Button_Switch_SMD:SW_SPDT_PCM12, F.Cu at (84.5, 48.0)
- added U1: STM32F103C8T6, Package_QFP:LQFP-48_7x7mm_P0.5mm, F.Cu at (95.2, 61.8)
- added U2: AMS1117-3.3, Package_TO_SOT_SMD:SOT-223-3_TabPin2, F.Cu at (104.0, 70.2)
- added Y1: 16MHz, Crystal:Crystal_SMD_3225-4Pin_3.2x2.5mm, F.Cu at (85.2, 61.6)
